File: C64 BlinkenDiag/C64 BlinkenDiag.kicad_pcb (KiCad board)
At the start: 2 copper layers, 99.4 x 99.9 mm, 64 parts, among them J1 C64-Exp-Port, J2 VOLTMETER, M1 Mounting, M2 Mounting, M3 Mounting, M4 Mounting, SW1 ROM_DIS, SW2 FUNCTION, SW3 ROM_BANK, SW4 RESET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

Commit message: Updated gerber files
Other:
- board text added: "C64 BlinkenDiag (rev. B) github.com/tebl"
- board text removed: "C64 BlinkenDiag (rev. A) github.com/tebl"
