File: C64 BlinkenDiag Faceplate/C64 BlinkenDiag Faceplate.kicad_pcb (KiCad board)
At the start: 2 copper layers, 99.4 x 70.1 mm, 4 parts, among them M1 Mounting, M2 Mounting, M3 Mounting, M4 Mounting

Commit message: Updated gerber files
Other:
- board text added: "R/~W"
- board text removed: "WRITE"
